File: ChargerControlBoard/DynamicBrakeGrid.kicad_pcb (KiCad board)
At the start: 4 copper layers, 175 x 125 mm, 111 parts, among them IC1 ISO1042BDWVR, IC5 LM358DR, IC6 MCP2515-e_ST, J1 1987724, J10 5442251, J11 5442251, J12 5442251, J13 38969-0002, J14 5442251, J15 5442251, J16 1987724, J17 1987724, J18 38969-0002, J2 1987724, J24 5442251, J25 5442251, J26 5442251, J27 5442251, J28 5442251, J3 1987724, J4 1987724, J5 5442251, J6 5442251, J7 5442251, J8 5442251, J9 5442251, M1 Fan_4pin, M2 Fan_4pin, M3 Fan_4pin, M8 Fan_4pin, Q1 SIHFR120-GE3, Y1 8MHz

Commit message: Finish Layout On Control Board
Parts:
- removed the G*** at (452.0, 114.0)
- added G***: LOGO, InverterCom:Char_NeilDylandy_20mm, F.Cu at (130.0, 64.0)
- moved G*** 401.4 mm to (92.0, 121.0)
- moved G*** 360.0 mm to (68.0, 123.0)
- moved H2 261.2 mm to (57.0, 124.0)
- moved J13 215.7 mm to (141.7, 139.8), turned to 90 degrees
- moved J18 176.6 mm to (141.7, 109.3), turned to 90 degrees
- moved R65 168.4 mm to (131.0, 144.0)
- moved R67 164.8 mm to (131.0, 125.0)
- moved R66 162.6 mm to (131.0, 135.0)
- moved R68 159.0 mm to (131.0, 116.0)
- moved R69 155.0 mm to (131.0, 107.0), turned to 90 degrees
- moved R70 141.9 mm to (131.0, 98.0), turned to -90 degrees
- moved J26 139.0 mm to (117.0, 113.0), turned to 90 degrees
- moved R71 134.1 mm to (132.0, 84.0), turned to 0 degrees
- moved C105 133.3 mm to (47.0, 82.0), turned to 180 degrees
- moved C69 131.7 mm to (131.9, 88.5), turned to 0 degrees
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Routing:
- net EVSE_CURRENT_PWM_INTERRUPT: track 0.00 -> 219.2 mm, vias 0 -> 3
- net +12V: track 112.1 -> 279.4 mm
- net LCD_SDA: track 0.00 -> 166.7 mm, vias 0 -> 2
- net LCD_SCL: track 0.00 -> 155.4 mm, vias 0 -> 3
- net +5V: track 157.6 -> 310.4 mm, vias 14 -> 16
- net Arduino_VInSense: track 239.2 -> 145.2 mm
- net Arduino_VoltageSetSense: track 0.00 -> 78.7 mm, vias 0 -> 1
- net Arduino_CurrentSetSense: track 0.00 -> 62.6 mm, vias 0 -> 1
- net EVSE_ENABLE: track 272.7 -> 220.6 mm, vias 3 -> 4
- net StatusLED_1: track 107.2 -> 156.5 mm, vias 4 -> 5
- net StatusLED_0: track 108.6 -> 148.7 mm, vias 4 -> 5
- net Arduino_LCDBacklightSense: track 61.6 -> 101.7 mm, vias 2 -> 3
- net GND: track 54.4 -> 17.3 mm, vias 500 -> 356
- net CanH_External: track 27.9 -> 62.6 mm, vias 3 -> 0
- net CanL_External: track 81.0 -> 60.8 mm
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- added copper zone on B.Cu, net DC_LINK_V+
Other:
- board text added: "GND AIN0 +5V"
- board text added: "GND AIN2 +5V"
- board text added: "GND AIN3 +5V"

Commit message: Update OBC Board
Routing:
- net +5V: track 310.4 -> 312.4 mm
- net GND: vias 356 -> 406
